Commit message: Update launch and URDF files to reflect project name change and enhance material definitions

File: urdf/gazebo_visual.xacro (robot description, xacro)
@@ -2,35 +2,71 @@
 <robot xmlns:xacro="http://www.ros.org/wiki/xacro">
     <gazebo reference="base_link">
-        <material>Gazebo/Green</material>
+        <material>
+            <ambient>0 1 0 1</ambient>
+            <diffuse>0 1 0 1</diffuse>
+            <specular>0.1 0.1 0.1 1</specular>
+        </material>
     </gazebo>
     <gazebo reference="fielder_chassis">
-        <material>Gazebo/White</material>
+        <material>
+            <ambient>0 0 1 1</ambient>
+            <diffuse>0 0 1 1</diffuse>
+            <specular>0.1 0.1 0.1 1</specular>
+        </material>
     </gazebo>
     <gazebo reference="lidar_link">
-        <material>Gazebo/Blue</material>
+        <material>
+            <ambient>0 0 1 1</ambient>
+            <diffuse>0 0 1 1</diffuse>
+            <specular>0.1 0.1 0.1 1</specular>
+        </material>
     </gazebo>
     <gazebo reference="left_wheel_link">
-        <material>Gazebo/Red</material>
+        <material>
+            <ambient>1 0 0 1</ambient>
+            <diffuse>1 0 0 1</diffuse>
+            <specular>0.1 0.1 0.1 1</specular>
+        </material>
     </gazebo>
     <gazebo reference="right_wheel_link">
-        <material>Gazebo/Red</material>
+        <material>
+            <ambient>1 0 0 1</ambient>
+            <diffuse>1 0 0 1</diffuse>
+            <specular>0.1 0.1 0.1 1</specular>
+        </material>
     </gazebo>
     <gazebo reference="castor_wheel_front_right">
-        <material>Gazebo/Black</material>
+        <material>
+            <ambient>0 0 0 1</ambient>
+            <diffuse>0 0 0 1</diffuse>
+            <specular>0.1 0.1 0.1 1</specular>
+        </material>
         <mu1 value="0.005"/>
         <mu2 value="0.005"/>
     </gazebo>
     <gazebo reference="castor_wheel_front_left">
-        <material>Gazebo/Black</material>
+        <material>
+            <ambient>0 0 0 1</ambient>
+            <diffuse>0 0 0 1</diffuse>
+            <specular>0.1 0.1 0.1 1</specular>
+        </material>
         <mu1 value="0.005"/>
         <mu2 value="0.005"/>
     </gazebo>
     <gazebo reference="castor_wheel_rear_right">
-        <material>Gazebo/Black</material>
+        <material>
+            <ambient>0 0 0 1</ambient>
+            <diffuse>0 0 0 1</diffuse>
+            <specular>0.1 0.1 0.1 1</specular>
+        </material>
         <mu1 value="0.005"/>
         <mu2 value="0.005"/>
     </gazebo>
     <gazebo reference="castor_wheel_rear_left">
-        <material>Gazebo/Black</material>
+        <material>
+            <ambient>0 0 0 1</ambient>
+            <diffuse>0 0 0 1</diffuse>
+            <specular>0.1 0.1 0.1 1</specular>
+        </material>
         <mu1 value="0.005"/>
         <mu2 value="0.005"/>
